File: ESP32-SSH-bridge.sch (KiCad schematic (older format))
At the start: 16 parts

Commit message: Initial commit of the version that takes a simple plug-in dev board
Parts:
- removed C? (x2): C_Small, symbol Device:C_Small
- removed C?: 0.1uF, symbol Device:C_Small
- removed C?: 4.7uF, symbol Device:C_Small
- removed D?: RED, symbol Device:LED_Small
- removed D?: GREEN, symbol Device:LED_Small
- removed J?: USB_B_Micro, symbol Connector:USB_B_Micro
- removed J?: Programmer, symbol Connector_Generic:Conn_01x06
- removed J?: Device, symbol Connector_Generic:Conn_01x06
- removed R? (x3): 1k, symbol Device:R_Small
- removed U?: ESP32-WROOM-32, symbol RF_Module:ESP32-WROOM-32
- removed U?: AZ1117-3.3, symbol Regulator_Linear:AZ1117-3.3
- removed U?: CP2102N-A01-GQFN24, Package_DFN_QFN:QFN-24-1EP_4x4mm_P0.5mm_EP2.6x2.6mm, symbol Interface_USB:CP2102N-A01-GQFN24
- added C1: 10uF, Capacitor_THT:CP_Radial_D6.3mm_P2.50mm, symbol Device:C_Small
- added J1, J2: Conn_01x07, Connector_PinSocket_2.54mm:PinSocket_1x07_P2.54mm_Vertical, symbol Connector_Generic:Conn_01x07
- added J4: +5V, Connector_PinHeader_2.54mm:PinHeader_1x02_P2.54mm_Horizontal, symbol Connector_Generic:Conn_01x02
- J3: renamed from J?; footprint (none) -> Connector_Dsub:DSUB-9_Female_Horizontal_P2.77x2.84mm_EdgePinOffset9.90mm_Housed_MountingHolesOffset11.32mm
Connections:
- net labels added: +3V3
- net labels removed: +3.3V
- wire segments 101 -> 31
Other:
- note added: "Dirty ESP32-dev"
